File: MC8P_MIDI_CONTROLLER_KiCad/MC8P_MIDI_CONTROLLER/MC8P_MIDI_CONTROLLER.kicad_pcb (KiCad board)
At the start: 2 copper layers, 155 x 288 mm, 61 parts, among them J1 MIDI OUT, SW1 ASSIGN, SW2 ENTER, SW3 PREV, SW4 NEXT, U1 Teensy4.0

Commit message: PCB Update
- Fixes power resets/brownouts
- disconnected POTS, BUTTONS and MIDI OUT from Vin
- connected POTS & BUTTONS to 3V3
- connected MIDI OUT to VUSB
Parts:
- removed C10: 100nF, Capacitor_THT:C_Disc_D5.0mm_W2.5mm_P5.00mm
- removed C11: 10uF, Capacitor_THT:C_Disc_D5.0mm_W2.5mm_P5.00mm
- removed C14: 100uF, Capacitor_THT:CP_Radial_D4.0mm_P1.50mm
Connections:
- C12 pad 1: Vcc -> 3V3
- C13 pad 1: Vcc -> 3V3
- C9 pad 1: Vcc -> 3V3
- RV1 pad 3: Vcc -> 3V3
- RV2 pad 3: Vcc -> 3V3
- RV3 pad 3: Vcc -> 3V3
- RV4 pad 3: Vcc -> 3V3
- RV5 pad 3: Vcc -> 3V3
- RV6 pad 3: Vcc -> 3V3
- RV7 pad 3: Vcc -> 3V3
- RV8 pad 3: Vcc -> 3V3
- SW1 pad 1: Vcc -> 3V3
- SW2 pad 1: Vcc -> 3V3
- SW3 pad 1: Vcc -> 3V3
- SW4 pad 1: Vcc -> 3V3
- U1 pad 33: Vcc -> unconnected-(U1-VIN-Pad33)
- U1 pad 34: unconnected-(U1-VUSB-Pad34) -> Vcc
Routing:
- net Vcc: track 528.5 -> 45.8 mm
- net 3V3: track 106.5 -> 554.3 mm
Other:
- board text added: ".axs instruments"
- board text removed: ".AXS INSTRUMENTS"
- board text removed: ".AXS Instruments"
- board text removed: "SNo."

Commit message: Schematic & PCB labelling update
Updated Capacitor labelling (C9-11)
Parts:
- renumbered C12 to C10, C13 to C11
Changed lines of the file:
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@@
 		(descr "C, Disc series, Radial, pin pitch=5.00mm, diameter*width=5*2.5mm^2, Capacitor, http://cdn-reichelt.de/documents/datenblatt/B300/DS_KERKO_TC.pdf")
 		(tags "C Disc series Radial pin pitch 5.00mm diameter 5mm width 2.5mm Capacitor")
-		(property "Reference" "C12"
+		(property "Reference" "C10"
 			(at 2.5 -2.5 90)
 			(layer "F.SilkS")
@@
 		(descr "CP, Radial series, Radial, pin pitch=1.50mm, diameter=4mm, height=7mm, Electrolytic Capacitor")
 		(tags "CP Radial series Radial pin pitch 1.50mm diameter 4mm height 7mm Electrolytic Capacitor")
-		(property "Reference" "C13"
+		(property "Reference" "C11"
 			(at -3 -0.5 90)
 			(layer "F.SilkS")

Commit message: PCB Updates
- Added dedicated 5V Centre Positive power input
- Added PCBWay logo for sponsor
- Updated UI Components with new Alagard font
Parts:
- added C12: 10uF_4x5.3_10V, Capacitor_THT:CP_Radial_D4.0mm_P1.50mm, F.Cu at (113.5, 31.8)
- added G***: LOGO, pcbWayLogo:pcbWay_LOGO_FSILK_15mm, F.Cu at (157.8, 290.0)
- added J2: 5V, Connector_BarrelJack:BarrelJack_GCT_DCJ200-10-A_Horizontal, F.Cu at (122.2, 35.5)
- R5, R6: value 10k_0402 -> 220R
Connections:
- U1 pad 33: unconnected-(U1-VIN-Pad33) -> 5V
Routing:
- net 5V: track 0.00 -> 61.4 mm
- net 3V3: track 554.3 -> 524.3 mm
Other:
- board text added: "5V DC in"
- board text added: "8 assignable potentiometers OLED Screen for UI Kailh Switches"
- board text removed: "8 assignable potentiometers OLED Screen for UI Cherry MX Switches"

Commit message: PCB Rev3
- STM32F411CEU6 Black Pill with
W25Q64 flash
- Added DC Jack for powering externally
- restructured KiCad Folder
- Added production folder with BOM
Parts:
- removed the ? at (169.0, 210.0)
- removed the ? at (169.0, 290.0)
- removed the ? at (26.0, 210.0)
- removed the ? at (169.0, 198.0)
- removed the ? at (26.0, 290.0)
- removed the ? at (26.0, 198.0)
- removed the ? at (26.0, 106.0)
- removed the ? at (169.0, 118.0)
- removed the ? at (26.0, 118.0)
- removed the G*** at (122.0, 229.1) (x2)
- removed the G*** at (112.5, 224.8)
- removed the REF** at (83.0, 161.3)
- removed the REF** at (106.0, 185.2)
- removed the REF** at (26.0, 26.0)
- removed the REF** at (106.0, 161.3)
- removed the REF** at (83.0, 185.2)
- removed the REF** at (169.0, 106.0)
- removed the REF** at (169.0, 26.0)
- removed the REF** at (60.0, 185.2)
- removed the REF** at (60.0, 161.3)
- removed the REF** at (37.0, 185.2)
- removed the REF** at (37.0, 161.3)
- added ?: , , F.Cu at (167.2, 120.5)
- added ?: , , F.Cu at (167.3, 212.5)
- added ?: , , F.Cu at (24.2, 108.5)
- added ?: , , F.Cu at (24.2, 120.5)
- added ?: , , F.Cu at (167.2, 200.5)
- added ?: , , F.Cu at (167.3, 292.5)
- added ?: , , F.Cu at (24.3, 212.5)
- added ?: , , F.Cu at (24.2, 200.5)
- added ?: , , F.Cu at (24.3, 292.5)
- added C13: 100nF_0603_16V, Capacitor_SMD:C_1206_3216Metric, F.Cu at (80.8, 30.8)
- added C14: 100nF_0603_16V, Capacitor_SMD:C_1206_3216Metric, F.Cu at (134.8, 33.5)
- added C15: 100nF_0603_16V, Capacitor_SMD:C_1206_3216Metric, F.Cu at (68.5, 68.9)
- added C16: 10uF, Capacitor_SMD:C_1206_3216Metric_Pad1.33x1.80mm_HandSolder, F.Cu at (71.0, 68.9)
- added D1: LED, LED_SMD:LED_1206_3216Metric_Pad1.42x1.75mm_HandSolder, F.Cu at (43.0, 53.8)
- added D2: BAT43, PCM_Diode_SMD_AKL:D_1206_3216Metric_Pad1.42x1.75mm_HandSolder, F.Cu at (70.0, 64.5)
- added G***: LOGO, MC8P_BITMAP_FOOTPRINTS:MC8P_PXLART_SPACE_FMASK_45X40, F.Cu at (110.8, 227.2)
- added G*** (x2): LOGO, MC8P_BITMAP_FOOTPRINTS:MC8P_PXLART_SPACE_FMASK_45X40, F.Cu at (120.3, 231.6)
- added R7: 10k_0402, PCM_4ms_Resistor:R_0603, F.Cu at (94.2, 29.5)
- added R8: 10k_0402, PCM_4ms_Resistor:R_0603, F.Cu at (42.2, 51.0)
- added REF**: Panel Knob 2P, SimpleSynthPanel:Panel Knob 2P, F.Cu at (58.3, 187.7)
- added REF**: MountingHole_M3_Standoff, DIYSynthMNL:MountingHole_M3_Standoff, F.Cu at (167.2, 28.5)
- added REF**: Panel Knob 2P, SimpleSynthPanel:Panel Knob 2P, F.Cu at (35.3, 163.8)
- added REF**: Panel Knob 2P, SimpleSynthPanel:Panel Knob 2P, F.Cu at (104.3, 163.8)
- added REF**: Panel Knob 2P, SimpleSynthPanel:Panel Knob 2P, F.Cu at (81.2, 163.8)
- added REF**: Panel Knob 2P, SimpleSynthPanel:Panel Knob 2P, F.Cu at (104.3, 187.7)
- added REF**: Panel Knob 2P, SimpleSynthPanel:Panel Knob 2P, F.Cu at (58.2, 163.8)
- added REF**: Panel Knob 2P, SimpleSynthPanel:Panel Knob 2P, F.Cu at (35.3, 187.7)
- added REF**: Panel Knob 2P, SimpleSynthPanel:Panel Knob 2P, F.Cu at (81.3, 187.7)
- added REF**: MountingHole_M3_Standoff, DIYSynthMNL:MountingHole_M3_Standoff, F.Cu at (24.2, 28.5)
- added REF**: MountingHole_M3_Standoff, DIYSynthMNL:MountingHole_M3_Standoff, F.Cu at (167.2, 108.5)
- added U3: CD74HC4067M, Package_SO:SOIC-24W_7.5x15.4mm_P1.27mm, F.Cu at (89.8, 37.2)
- added U4: W25Q64, Package_SO:SOIC-8_3.9x4.9mm_P1.27mm, F.Cu at (37.1, 47.9)
- C1, C2, C3, C4, C5, C6, C7, C8: footprint Capacitor_THT:C_Axial_L3.8mm_D2.6mm_P7.50mm_Horizontal -> Capacitor_SMD:C_1206_3216Metric_Pad1.33x1.80mm_HandSolder
- C10, C9: footprint Capacitor_THT:C_Disc_D5.0mm_W2.5mm_P5.00mm -> Capacitor_SMD:C_1206_3216Metric_Pad1.33x1.80mm_HandSolder
- C12: value 10uF_4x5.3_10V -> 100nF_0603_16V; footprint Capacitor_THT:CP_Radial_D4.0mm_P1.50mm -> Capacitor_SMD:C_1206_3216Metric
- J1: moved to B.Cu
- J2: value 5V -> Jack-DC
- R1, R2, R3, R4: value 10k_0402 -> 10k; footprint PCM_4ms_Resistor:R_Axial_DIN0207_L6.3mm_D2.5mm_P7.62mm_Horizontal -> PCM_4ms_Resistor:R_0603
- R5, R6: value 220R -> 33R; footprint PCM_4ms_Resistor:R_Axial_DIN0207_L6.3mm_D2.5mm_P7.62mm_Horizontal -> PCM_4ms_Resistor:R_0603
- U1: value Teensy4.0 -> ~; footprint teensy:Teensy40 -> blackpill:Z_module_black_pill_STM32F411; moved to B.Cu
- moved C5 80.6 mm to (37.2, 85.5), turned to 0 degrees
- moved C12 78.8 mm to (37.6, 53.1), turned to 0 degrees
- moved C6 56.7 mm to (59.8, 85.8), turned to 0 degrees
- moved C11 52.8 mm to (56.0, 28.2), turned to 0 degrees
- moved C10 45.7 mm to (57.5, 34.8), turned to 0 degrees
- moved C9 40.8 mm to (57.5, 32.0), turned to 0 degrees
- moved C1 40.1 mm to (36.8, 61.5), turned to 0 degrees
- moved C7 37.3 mm to (82.8, 85.5), turned to 0 degrees
- moved C8 33.9 mm to (105.7, 85.5), turned to 0 degrees
- moved R4 31.4 mm to (119.5, 71.2)
- moved R3 25.6 mm to (119.5, 69.5)
- moved C2 22.9 mm to (59.8, 61.5), turned to 0 degrees
- moved R2 18.2 mm to (119.5, 66.0)
- moved C4 17.4 mm to (106.0, 61.8), turned to 0 degrees
- moved R1 15.9 mm to (119.5, 67.8)
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Connections:
- C1 pad 1: A0 -> pot1
- C12 pad 1: 5V -> GND
- C12 pad 2: GND -> 3V3
- C2 pad 1: A1 -> pot2
- C3 pad 1: A2 -> pot3
- C4 pad 1: A3 -> pot4
- C5 pad 1: A9 -> pot5
- C6 pad 1: A8 -> pot6
- C7 pad 1: A7 -> pot7
- C8 pad 1: A6 -> pot8
- J2 pad 1: 5V -> Net-(D2-A)
- R1 pad 1: D5 -> ASSIGN
- R2 pad 1: D6 -> ENTER
- R3 pad 1: D7 -> PREV
- R4 pad 1: D8 -> NEXT
- R6 pad 1: Vcc -> 3V3
- RV1 pad 2: A0 -> pot1
- RV2 pad 2: A1 -> pot2
- RV3 pad 2: A2 -> pot3
- RV4 pad 2: A3 -> pot4
- RV5 pad 2: A6 -> pot5
- RV6 pad 2: A7 -> pot6
- RV7 pad 2: A8 -> pot7
- RV8 pad 2: A9 -> pot8
- SW1 pad 2: D5 -> ASSIGN
- SW2 pad 2: D6 -> ENTER
- SW3 pad 2: D7 -> PREV
- SW4 pad 2: D8 -> NEXT
- U1 pad 1: GND -> ASSIGN
- U1 pad 10: D8 -> unconnected-(U1-PA15-Pad10)
- U1 pad 14: unconnected-(U1-12_MISO_MQSL-Pad14) -> SCL0
- U1 pad 15: unconnected-(U1-VBAT-Pad15) -> SDA0
- U1 pad 17: GND -> unconnected-(U1-1PB9-Pad17)
- U1 pad 18: unconnected-(U1-PROGRAM-Pad18) -> Vcc
- U1 pad 19: unconnected-(U1-ON_OFF-Pad19) -> GND
- U1 pad 2: unconnected-(U1-0_RX1_CRX2_CS1-Pad2) -> ENTER
- U1 pad 20: unconnected-(U1-13_SCK_CRX1_LED-Pad20) -> 3V3
- U1 pad 21: A0 -> unconnected-(U1-VBAT-Pad21)
- U1 pad 22: A1 -> unconnected-(U1-PC13-Pad22)
- U1 pad 23: A2 -> unconnected-(U1-PC14-Pad23)
- U1 pad 24: A3 -> unconnected-(U1-PC15-Pad24)
- U1 pad 25: SDA0 -> unconnected-(U1-RESET-Pad25)
- U1 pad 26: SCL0 -> unconnected-(U1-PA0/ADC0-Pad26)
- U1 pad 27: A6 -> SIG
- U1 pad 28: A7 -> TX0
- U1 pad 29: A8 -> unconnected-(U1-PA3/ADC3/RX2-Pad29)
- U1 pad 3: TX0 -> PREV
- U1 pad 30: A9 -> CS
- U1 pad 31: 3V3 -> CLK
- U1 pad 32: GND -> MISO
- U1 pad 33: 5V -> MOSI
- U1 pad 34: Vcc -> unconnected-(U1-PB0/ADC8-Pad34)
- U1 pad 38: unconnected-(U1-27_A13_SCK1-Pad38) -> 3V3
- U1 pad 39: unconnected-(U1-28_RX7-Pad39) -> GND
- U1 pad 4: unconnected-(U1-2_OUT2-Pad4) -> NEXT
- U1 pad 40: unconnected-(U1-29_TX7-Pad40) -> Vcc
- U1 pad 5: unconnected-(U1-3_LRCLK2-Pad5) -> S0
- U1 pad 6: unconnected-(U1-4_BCLK2-Pad6) -> S1
- U1 pad 7: D5 -> S2
- U1 pad 8: D6 -> S3
- U1 pad 9: D7 -> unconnected-(U1-PA12-Pad9)
Routing:
- net D5: track 278.5 -> 0.00 mm
- net D7: track 257.8 -> 0.00 mm
- net D6: track 252.4 -> 0.00 mm
- net D8: track 250.9 -> 0.00 mm
- net NEXT: track 0.00 -> 208.8 mm, vias 0 -> 1
- net PREV: track 0.00 -> 198.1 mm, vias 0 -> 1
- net A6: track 158.7 -> 0.00 mm
- net Net-(D2-A): track 0.00 -> 157.3 mm, vias 0 -> 1
- net pot1: track 0.00 -> 152.4 mm, vias 0 -> 1
- net ENTER: track 0.00 -> 148.3 mm, vias 0 -> 1
- net pot5: track 0.00 -> 141.4 mm, vias 0 -> 2
- net A7: track 136.6 -> 0.00 mm
- net pot2: track 0.00 -> 132.2 mm, vias 0 -> 3
- net pot6: track 0.00 -> 124.2 mm, vias 0 -> 2
- net A8: track 115.3 -> 0.00 mm
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
Commit message: PCB revisions
Parts:
- R5, R6: value 33R -> 220R
Connections:
- J2 pad 3: GND -> (no net)
- U1 pad 10: unconnected-(U1-PA15-Pad10) -> S3
- U1 pad 8: S3 -> unconnected-(U1-PA11-Pad8)
Routing:
- net GND: track 34.3 -> 54.9 mm, vias 16 -> 17
- net S3: track 114.5 -> 109.3 mm
- net pot2: track 132.2 -> 135.0 mm
- net pot1: track 152.4 -> 155.2 mm
Changed lines of the file:
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@@
 	(net 45 "unconnected-(U1-PB0{slash}ADC8-Pad34)")
 	(net 46 "unconnected-(U1-PB4{slash}SCL2-Pad12)")
-	(net 47 "unconnected-(U1-PA15-Pad10)")
+	(net 47 "unconnected-(U1-PA11-Pad8)")
 	(net 48 "unconnected-(U1-PB8-Pad16)")
 	(net 49 "unconnected-(U1-PC13-Pad22)")
@@
 			)
 		)
-		(property "Value" "33R"
+		(property "Value" "220R"
 			(at -1 -1.25 0)
 			(layer "F.SilkS")
@@
 			(layers "*.Cu" "*.Mask")
 			(remove_unused_layers no)
-			(net 2 "GND")
 		)
 		(embedded_fonts no)
@@
 			)
 		)
+		(property ki_fp_filters "C_*")
+		(sheetname "/")
+		(sheetfile "MC8P_MIDI_CONTROLLER.kicad_sch")
 		(attr smd)
 		(fp_line
@@
 			)
 		)
+		(property ki_fp_filters "C_*")
+		(sheetname "/")
+		(sheetfile "MC8P_MIDI_CONTROLLER.kicad_sch")
 		(attr smd)
 		(fp_line
@@
 			)
 		)
-		(property "Value" "33R"
+		(property "Value" "220R"
 			(at 0.75 -1.25 0)
 			(layer "F.SilkS")
@@
 			(layers "*.Cu" "*.Mask")
 			(remove_unused_layers no)
-			(net 25 "S3")
+			(net 47 "unconnected-(U1-PA11-Pad8)")
 			(pinfunction "PA11")
 			(pintype "bidirectional")
@@
 			(layers "*.Cu" "*.Mask")
 			(remove_unused_layers no)
-			(net 47 "unconnected-(U1-PA15-Pad10)")
+			(net 25 "S3")
 			(pinfunction "PA15")
 			(pintype "bidirectional")
@@
 	)
 	(segment
+		(start 35.25 61.5)
+		(end 35.25 64.2815)
+		(width 0.5)
+		(layer "F.Cu")
+		(net 1)
+	)
+	(segment
 		(start 92.925 41.9)
 		(end 92.925 47.175)
@@
 	)
 	(segment
+		(start 94.25 28.65)
+		(end 91.9 28.65)
+		(width 0.5)
+		(layer "F.Cu")
+		(net 2)
+	)
+	(segment
 		(start 38.8125 85.5)
 		(end 40.5 85.5)
@@
 	)
 	(segment
-		(start 94.25 28.65)
-		(end 94.25 27.5)
+		(start 91.9 28.65)
+		(end 91.75 28.5)
 		(width 0.5)
 		(layer "F.Cu")
@@
 	)
 	(via
+		(at 76.75 48)
+		(size 0.6)
+		(drill 0.3)
+		(layers "F.Cu" "B.Cu")
+		(net 2)
+	)
+	(via
 		(at 68.25 71.6875)
 		(size 0.6)
@@
 	)
 	(via
-		(at 94.25 27.5)
+		(at 91.75 28.5)
 		(size 0.6)
 		(drill 0.3)
@@
 	)
 	(segment
+		(start 83.7527 64.2842)
+		(end 83.7527 55.0027)
+		(width 0.5)
+		(layer "B.Cu")
+		(net 2)
+	)
+	(segment
+		(start 83.7527 55.0027)
+		(end 76.75 48)
+		(width 0.5)
+		(layer "B.Cu")
+		(net 2)
+	)
+	(segment
+		(start 58.1875 64.219)
+		(end 58.2527 64.2842)
+		(width 0.5)
+		(layer "F.Cu")
+		(net 3)
+	)
+	(segment
 		(start 58 78.5)
 		(end 58 80.25)
@@
 	)
 	(segment
+		(start 58.1875 61.5)
+		(end 58.1875 64.219)
+		(width 0.5)
+		(layer "F.Cu")
+		(net 3)
+	)
+	(segment
 		(start 92.5 49.5)
 		(end 98.75 49.5)
@@
 	)
 	(segment
-		(start 144.87 30.805)
-		(end 141.925 33.75)
+		(start 114.75 27)
+		(end 85.5 27)
 		(width 0.5)
 		(layer "B.Cu")
@@
 	)
 	(segment
-		(start 74 32.25)
-		(end 72.75 33.5)
+		(start 144.87 30.805)
+		(end 141.925 33.75)
 		(width 0.5)
 		(layer "B.Cu")
@@
 	)
 	(segment
-		(start 80.25 32.25)
-		(end 74 32.25)
+		(start 141.925 33.75)
+		(end 121.5 33.75)
 		(width 0.5)
 		(layer "B.Cu")
@@
 	)
 	(segment
-		(start 141.925 33.75)
-		(end 121.5 33.75)
+		(start 74 32.25)
+		(end 72.75 33.5)
 		(width 0.5)
 		(layer "B.Cu")
@@
 	)
 	(segment
-		(start 115 27.25)
-		(end 85.25 27.25)
+		(start 80.25 32.25)
+		(end 74 32.25)
 		(width 0.5)
 		(layer "B.Cu")
@@
 	)
 	(segment
-		(start 121.5 33.75)
-		(end 115 27.25)
+		(start 85.5 27)
+		(end 80.25 32.25)
 		(width 0.5)
 		(layer "B.Cu")
@@
 	)
 	(segment
-		(start 85.25 27.25)
-		(end 80.25 32.25)
+		(start 121.5 33.75)
+		(end 114.75 27)
 		(width 0.5)
 		(layer "B.Cu")
@@
 	)
 	(segment
-		(start 70.15 42.15)
-		(end 65.87 42.15)
+		(start 92.5 80.75)
+		(end 74.75 80.75)
 		(width 0.5)
 		(layer "B.Cu")
@@
 	)
 	(segment
-		(start 92.5 80.75)
-		(end 74.75 80.75)
+		(start 97.25 34.5)
+		(end 99.25 36.5)
 		(width 0.5)
 		(layer "B.Cu")
@@
 	(segment
 		(start 71.25 77.25)
-		(end 71.25 43.25)
+		(end 71.25 48.5)
 		(width 0.5)
 		(layer "B.Cu")
@@
 	)
 	(segment
-		(start 99.25 36.5)
-		(end 99.25 45)
+		(start 74.75 80.75)
+		(end 71.25 77.25)
 		(width 0.5)
 		(layer "B.Cu")
@@
 	)
 	(segment
-		(start 74.75 80.75)
-		(end 71.25 77.25)
+		(start 71.25 48.5)
+		(end 70 47.25)
 		(width 0.5)
 		(layer "B.Cu")
@@
 	)
 	(segment
-		(start 97.25 34.5)
-		(end 99.25 36.5)
+		(start 99.25 45)
+		(end 97 47.25)
 		(width 0.5)
 		(layer "B.Cu")
@@
 	)
 	(segment
-		(start 97 47.25)
-		(end 97 76.25)
+		(start 70 47.25)
+		(end 65.89 47.25)
 		(width 0.5)
 		(layer "B.Cu")
@@
 	)
 	(segment
-		(start 71.25 43.25)
-		(end 70.15 42.15)
+		(start 97 47.25)
+		(end 97 76.25)
 		(width 0.5)
 		(layer "B.Cu")
@@
 	)
 	(segment
-		(start 99.25 45)
-		(end 97 47.25)
+		(start 99.25 36.5)
+		(end 99.25 45)
+		(width 0.5)
+		(layer "B.Cu")
+		(net 25)
+	)
+	(segment
+		(start 65.89 47.25)
+		(end 65.87 47.23)
 		(width 0.5)
 		(layer "B.Cu")

Commit message: pcb revisions
Parts:
- D2: footprint PCM_Diode_SMD_AKL:D_1206_3216Metric_Pad1.42x1.75mm_HandSolder -> Diode_SMD:D_SOD-123
Changed lines of the file:
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@@
 		(embedded_fonts no)
 	)
-	(footprint "PCM_Diode_SMD_AKL:D_1206_3216Metric_Pad1.42x1.75mm_HandSolder"
+	(footprint "Diode_SMD:D_SOD-123"
 		(layer "F.Cu")
 		(at 70 64.5)
-		(descr "Diode SMD 1206 (3216 Metric), square (rectangular) end terminal, IPC_7351 nominal, (Body size source: http://www.tortai-tech.com/upload/download/2011102023233369053.pdf), Alternate KiCad Library")
-		(tags "diode 1206 handsolder")
+		(descr "SOD-123")
+		(tags "SOD-123")
 		(property "Reference" "D2"
-			(at 0 -2.159 0)
+			(at 0 -2 0)
 			(layer "F.SilkS")
 			(effects
@@
 		)
 		(property "Value" "BAT43"
-			(at 0 1.82 0)
+			(at 0 2.1 0)
 			(layer "F.Fab")
 			(effects
@@
 		(property "Datasheet" "https://www.tme.eu/Document/1036f59816f6cf6d50674da5bd8b8c1f/BAT42.pdf"
 			(at 0 0 0)
+			(unlocked yes)
 			(layer "F.Fab")
 			(hide yes)
@@
 		(property "Description" "DO-35 Schottky diode, 30V, 200mA, Alternate KiCAD Library"
 			(at 0 0 0)
+			(unlocked yes)
 			(layer "F.Fab")
 			(hide yes)
@@
 		(attr smd)
 		(fp_line
-			(start -2.413 -1.143)
-			(end -2.413 1.143)
+			(start -2.36 -1)
+			(end -2.36 1)
 			(stroke
 				(width 0.12)
@@
 		)
 		(fp_line
-			(start -2.413 1.143)
-			(end 2.413 1.143)
+			(start -2.36 -1)
+			(end 1.65 -1)
 			(stroke
 				(width 0.12)
@@
 		)
 		(fp_line
-			(start -0.381 -0.635)
-			(end -0.381 0.635)
+			(start -2.36 1)
+			(end 1.65 1)
 			(stroke
 				(width 0.12)
@@
 		)
 		(fp_line
-			(start 2.413 -1.143)
-			(end -2.413 -1.143)
-			(stroke
-				(width 0.12)
-				(type solid)
-			)
-			(layer "F.SilkS")
-		)
-		(fp_line
-			(start 2.413 1.143)
-			(end 2.413 -1.143)
-			(stroke
-				(width 0.12)
-				(type solid)
-			)
-			(layer "F.SilkS")
-		)
-		(fp_poly
-			(pts
-				(xy 0.381 0.635) (xy -0.381 0) (xy 0.381 -0.635)
-			)
-			(stroke
-				(width 0.1)
-				(type solid)
-			)
-			(fill yes)
-			(layer "F.SilkS")
-		)
-		(fp_poly
-			(pts
-				(xy -0.3175 -1.143) (xy -1.27 -1.143) (xy -1.27 -1.397) (xy -0.3175 -1.397)
-			)
-			(stroke
-				(width 0.1)
-				(type solid)
-			)
-			(fill yes)
-			(layer "F.SilkS")
-		)
-		(fp_poly
-			(pts
-				(xy -0.3175 1.397) (xy -1.27 1.397) (xy -1.27 1.143) (xy -0.3175 1.143)
-			)
-			(stroke
-				(width 0.1)
-				(type solid)
-			)
-			(fill yes)
-			(layer "F.SilkS")
-		)
-		(fp_line
-			(start -2.4765 -1.4605)
-			(end 2.4765 -1.4605)
-			(stroke
-				(width 0.05)
-				(type solid)
-			)
-			(layer "F.CrtYd")
-		)
-		(fp_line
-			(start -2.4765 1.4605)
-			(end -2.4765 -1.4605)
-			(stroke
-				(width 0.05)
-				(type solid)
-			)
-			(layer "F.CrtYd")
-		)
-		(fp_line
-			(start 2.4765 -1.4605)
-			(end 2.4765 1.4605)
-			(stroke
-				(width 0.05)
-				(type solid)
-			)
-			(layer "F.CrtYd")
-		)
-		(fp_line
-			(start 2.4765 1.4605)
-			(end -2.4765 1.4605)
-			(stroke
-				(width 0.05)
-				(type solid)
-			)
-			(layer "F.CrtYd")
-		)
-		(fp_line
-			(start -1.6 -0.4)
-			(end -1.6 0.8)
-			(stroke
-				(width 0.1)
-				(type solid)
-			)
-			(layer "F.Fab")
-		)
-		(fp_line
-			(start -1.6 0.8)
-			(end 1.6 0.8)
-			(stroke
-				(width 0.1)
-				(type solid)
-			)
-			(layer "F.Fab")
-		)
-		(fp_line
-			(start -1.2 -0.8)
-			(end -1.6 -0.4)
-			(stroke
-				(width 0.1)
-				(type solid)
-			)
-			(layer "F.Fab")
-		)
-		(fp_line
-			(start 1.6 -0.8)
-			(end -1.2 -0.8)
-			(stroke
-				(width 0.1)
-				(type solid)
-			)
-			(layer "F.Fab")
-		)
-		(fp_line
-			(start 1.6 0.8)
-			(end 1.6 -0.8)
+			(start -2.35 -1.15)
+			(end -2.35 1.15)
+			(stroke
+				(width 0.05)
+				(type solid)
+			)
+			(layer "F.CrtYd")
+		)
+		(fp_line
+			(start -2.35 -1.15)
+			(end 2.35 -1.15)
+			(stroke
+				(width 0.05)
+				(type solid)
+			)
+			(layer "F.CrtYd")
+		)
+		(fp_line
+			(start 2.35 -1.15)
+			(end 2.35 1.15)
+			(stroke
+				(width 0.05)
+				(type solid)
+			)
+			(layer "F.CrtYd")
+		)
+		(fp_line
+			(start 2.35 1.15)
+			(end -2.35 1.15)
+			(stroke
+				(width 0.05)
+				(type solid)
+			)
+			(layer "F.CrtYd")
+		)
+		(fp_line
+			(start -1.4 -0.9)
+			(end 1.4 -0.9)
+			(stroke
+				(width 0.1)
+				(type solid)
+			)
+			(layer "F.Fab")
+		)
+		(fp_line
+			(start -1.4 0.9)
+			(end -1.4 -0.9)
+			(stroke
+				(width 0.1)
+				(type solid)
+			)
+			(layer "F.Fab")
+		)
+		(fp_line
+			(start -0.75 0)
+			(end -0.35 0)
+			(stroke
+				(width 0.1)
+				(type solid)
+			)
+			(layer "F.Fab")
+		)
+		(fp_line
+			(start -0.35 0)
+			(end -0.35 -0.55)
+			(stroke
+				(width 0.1)
+				(type solid)
+			)
+			(layer "F.Fab")
+		)
+		(fp_line
+			(start -0.35 0)
+			(end -0.35 0.55)
+			(stroke
+				(width 0.1)
+				(type solid)
+			)
+			(layer "F.Fab")
+		)
+		(fp_line
+			(start -0.35 0)
+			(end 0.25 -0.4)
+			(stroke
+				(width 0.1)
+				(type solid)
+			)
+			(layer "F.Fab")
+		)
+		(fp_line
+			(start 0.25 -0.4)
+			(end 0.25 0.4)
+			(stroke
+				(width 0.1)
+				(type solid)
+			)
+			(layer "F.Fab")
+		)
+		(fp_line
+			(start 0.25 0)
+			(end 0.75 0)
+			(stroke
+				(width 0.1)
+				(type solid)
+			)
+			(layer "F.Fab")
+		)
+		(fp_line
+			(start 0.25 0.4)
+			(end -0.35 0)
+			(stroke
+				(width 0.1)
+				(type solid)
+			)
+			(layer "F.Fab")
+		)
+		(fp_line
+			(start 1.4 -0.9)
+			(end 1.4 0.9)
+			(stroke
+				(width 0.1)
+				(type solid)
+			)
+			(layer "F.Fab")
+		)
+		(fp_line
+			(start 1.4 0.9)
+			(end -1.4 0.9)
 			(stroke
 				(width 0.1)
@@
 		)
 		(fp_text user "${REFERENCE}"
-			(at 0 0 0)
-			(layer "F.Fab")
-			(effects
-				(font
-					(size 0.8 0.8)
-					(thickness 0.12)
+			(at 0 -2 0)
+			(layer "F.Fab")
+			(effects
+				(font
+					(size 1 1)
+					(thickness 0.15)
 				)
 			)
 		)
 		(pad "1" smd roundrect
-			(at -1.4875 0)
-			(size 1.425 1.75)
+			(at -1.65 0)
+			(size 0.9 1.2)
 			(layers "F.Cu" "F.Mask" "F.Paste")
-			(roundrect_rratio 0.175439)
+			(roundrect_rratio 0.25)
 			(net 56 "Vcc")
 			(pinfunction "K")
@@
 		)
 		(pad "2" smd roundrect
-			(at 1.4875 0)
-			(size 1.425 1.75)
+			(at 1.65 0)
+			(size 0.9 1.2)
 			(layers "F.Cu" "F.Mask" "F.Paste")
-			(roundrect_rratio 0.175439)
+			(roundrect_rratio 0.25)
 			(net 38 "Net-(D2-A)")
 			(pinfunction "A")
@@
 		)
 		(embedded_fonts no)
-		(model "${KISYS3DMOD}/Diode_SMD.3dshapes/D_1206_3216Metric.wrl"
+		(model "${KICAD9_3DMODEL_DIR}/Diode_SMD.3dshapes/D_SOD-123.step"
 			(offset
 				(xyz 0 0 0)
