File: MC8P_MIDI_CONTROLLER_KiCad/MC8P_MIDI_CONTROLLER/MC8P_MIDI_CONTROLLER.kicad_pcb (KiCad board)
At the start: 2 copper layers, 155 x 288 mm, 71 parts, among them J1 MIDI OUT, J2 Jack-DC, SW1 ASSIGN, SW2 ENTER, SW3 PREV, SW4 NEXT, U3 CD74HC4067M, U4 W25Q64

Commit message: Mk1 PCB
Parts:
- removed the ? at (167.2, 120.5)
- removed the ? at (167.3, 212.5)
- removed the ? at (24.2, 108.5)
- removed the ? at (24.2, 120.5)
- removed the ? at (167.2, 200.5)
- removed the ? at (167.3, 292.5)
- removed the ? at (24.3, 212.5)
- removed the ? at (24.2, 200.5)
- removed the ? at (24.3, 292.5)
- removed C13, C14, C15: 100nF_0603_16V, Capacitor_SMD:C_1206_3216Metric
- removed C16: 10uF, Capacitor_SMD:C_1206_3216Metric_Pad1.33x1.80mm_HandSolder
- removed D1: LED, LED_SMD:LED_1206_3216Metric_Pad1.42x1.75mm_HandSolder
- removed D2: BAT43, Diode_SMD:D_SOD-123
- removed the G*** at (110.8, 227.2)
- removed the G*** at (120.3, 231.6) (x2)
- removed R7, R8: 10k_0402, PCM_4ms_Resistor:R_0603
- removed the REF** at (58.3, 187.7)
- removed the REF** at (167.2, 28.5)
- removed the REF** at (35.3, 163.8)
- removed the REF** at (104.3, 163.8)
- removed the REF** at (81.2, 163.8)
- removed the REF** at (104.3, 187.7)
- removed the REF** at (58.2, 163.8)
- removed the REF** at (35.3, 187.7)
- removed the REF** at (81.3, 187.7)
- removed the REF** at (24.2, 28.5)
- removed the REF** at (167.2, 108.5)
- removed U3: CD74HC4067M, Package_SO:SOIC-24W_7.5x15.4mm_P1.27mm
- removed U4: W25Q64, Package_SO:SOIC-8_3.9x4.9mm_P1.27mm
- added ?: , , F.Cu at (169.0, 210.0)
- added ?: , , F.Cu at (169.0, 290.0)
- added ?: , , F.Cu at (26.0, 210.0)
- added ?: , , F.Cu at (169.0, 198.0)
- added ?: , , F.Cu at (26.0, 290.0)
- added ?: , , F.Cu at (26.0, 198.0)
- added ?: , , F.Cu at (26.0, 106.0)
- added ?: , , F.Cu at (169.0, 118.0)
- added ?: , , F.Cu at (26.0, 118.0)
- added G*** (x2): LOGO, MC8P_BITMAP_FOOTPRINTS:MC8P_PXLART_SPACE_FMASK_45X40, F.Cu at (122.0, 229.1)
- added G***: LOGO, MC8P_BITMAP_FOOTPRINTS:MC8P_PXLART_SPACE_FMASK_45X40, F.Cu at (112.5, 224.8)
- added REF**: Panel Knob 2P, SimpleSynthPanel:Panel Knob 2P, F.Cu at (83.0, 161.3)
- added REF**: Panel Knob 2P, SimpleSynthPanel:Panel Knob 2P, F.Cu at (106.0, 185.2)
- added REF**: MountingHole_M3_Standoff, DIYSynthMNL:MountingHole_M3_Standoff, F.Cu at (26.0, 26.0)
- added REF**: Panel Knob 2P, SimpleSynthPanel:Panel Knob 2P, F.Cu at (106.0, 161.3)
- added REF**: Panel Knob 2P, SimpleSynthPanel:Panel Knob 2P, F.Cu at (83.0, 185.2)
- added REF**: MountingHole_M3_Standoff, DIYSynthMNL:MountingHole_M3_Standoff, F.Cu at (169.0, 106.0)
- added REF**: MountingHole_M3_Standoff, DIYSynthMNL:MountingHole_M3_Standoff, F.Cu at (169.0, 26.0)
- added REF**: Panel Knob 2P, SimpleSynthPanel:Panel Knob 2P, F.Cu at (60.0, 185.2)
- added REF**: Panel Knob 2P, SimpleSynthPanel:Panel Knob 2P, F.Cu at (60.0, 161.3)
- added REF**: Panel Knob 2P, SimpleSynthPanel:Panel Knob 2P, F.Cu at (37.0, 185.2)
- added REF**: Panel Knob 2P, SimpleSynthPanel:Panel Knob 2P, F.Cu at (37.0, 161.3)
- C1, C2, C3, C4, C5, C6, C7, C8: footprint Capacitor_SMD:C_1206_3216Metric_Pad1.33x1.80mm_HandSolder -> Capacitor_THT:C_Axial_L3.8mm_D2.6mm_P7.50mm_Horizontal
- C10, C9: footprint Capacitor_SMD:C_1206_3216Metric_Pad1.33x1.80mm_HandSolder -> Capacitor_THT:C_Disc_D5.0mm_W2.5mm_P5.00mm
- C12: value 100nF_0603_16V -> 10uF_4x5.3_10V; footprint Capacitor_SMD:C_1206_3216Metric -> Capacitor_THT:CP_Radial_D4.0mm_P1.50mm
- J1: moved to F.Cu
- J2: value Jack-DC -> 5V
- R1, R2, R3, R4: value 10k -> 10k_0402; footprint PCM_4ms_Resistor:R_0603 -> PCM_4ms_Resistor:R_Axial_DIN0207_L6.3mm_D2.5mm_P7.62mm_Horizontal
- R5, R6: footprint PCM_4ms_Resistor:R_0603 -> PCM_4ms_Resistor:R_Axial_DIN0207_L6.3mm_D2.5mm_P7.62mm_Horizontal
- U1: value ~ -> Teensy4.0; footprint blackpill:Z_module_black_pill_STM32F411 -> teensy:Teensy40; moved to F.Cu
- moved C5 80.6 mm to (111.0, 53.0), turned to 90 degrees
- moved C12 78.8 mm to (113.5, 31.8), turned to 90 degrees
- moved C6 56.7 mm to (106.0, 53.0), turned to 90 degrees
- moved C11 52.8 mm to (108.5, 33.8), turned to -90 degrees
- moved C10 45.7 mm to (103.0, 30.8), turned to -90 degrees
- moved C9 40.8 mm to (98.2, 30.8), turned to -90 degrees
- moved C1 40.1 mm to (76.0, 53.0), turned to 90 degrees
- moved C7 37.3 mm to (101.0, 53.0), turned to 90 degrees
- moved C8 33.9 mm to (96.0, 53.0), turned to 90 degrees
- moved R4 31.4 mm to (122.2, 40.0)
- moved R3 25.6 mm to (122.2, 44.0)
- moved C2 22.9 mm to (81.0, 53.0), turned to 90 degrees
- moved R2 18.2 mm to (122.2, 48.0)
- moved C4 17.4 mm to (91.0, 53.0), turned to 90 degrees
- moved R1 15.9 mm to (122.2, 52.1)
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Connections:
- C1 pad 1: pot1 -> A0
- C12 pad 1: GND -> 5V
- C12 pad 2: 3V3 -> GND
- C2 pad 1: pot2 -> A1
- C3 pad 1: pot3 -> A2
- C4 pad 1: pot4 -> A3
- C5 pad 1: pot5 -> A9
- C6 pad 1: pot6 -> A8
- C7 pad 1: pot7 -> A7
- C8 pad 1: pot8 -> A6
- J2 pad 1: Net-(D2-A) -> 5V
- J2 pad 3: (no net) -> GND
- R1 pad 1: ASSIGN -> D5
- R2 pad 1: ENTER -> D6
- R3 pad 1: PREV -> D7
- R4 pad 1: NEXT -> D8
- R6 pad 1: 3V3 -> Vcc
- RV1 pad 2: pot1 -> A0
- RV2 pad 2: pot2 -> A1
- RV3 pad 2: pot3 -> A2
- RV4 pad 2: pot4 -> A3
- RV5 pad 2: pot5 -> A6
- RV6 pad 2: pot6 -> A7
- RV7 pad 2: pot7 -> A8
- RV8 pad 2: pot8 -> A9
- SW1 pad 2: ASSIGN -> D5
- SW2 pad 2: ENTER -> D6
- SW3 pad 2: PREV -> D7
- SW4 pad 2: NEXT -> D8
- U1 pad 1: ASSIGN -> GND
- U1 pad 10: S3 -> D8
- U1 pad 14: SCL0 -> unconnected-(U1-12_MISO_MQSL-Pad14)
- U1 pad 15: SDA0 -> unconnected-(U1-VBAT-Pad15)
- U1 pad 17: unconnected-(U1-1PB9-Pad17) -> GND
- U1 pad 18: Vcc -> unconnected-(U1-PROGRAM-Pad18)
- U1 pad 19: GND -> unconnected-(U1-ON_OFF-Pad19)
- U1 pad 2: ENTER -> unconnected-(U1-0_RX1_CRX2_CS1-Pad2)
- U1 pad 20: 3V3 -> unconnected-(U1-13_SCK_CRX1_LED-Pad20)
- U1 pad 21: unconnected-(U1-VBAT-Pad21) -> A0
- U1 pad 22: unconnected-(U1-PC13-Pad22) -> A1
- U1 pad 23: unconnected-(U1-PC14-Pad23) -> A2
- U1 pad 24: unconnected-(U1-PC15-Pad24) -> A3
- U1 pad 25: unconnected-(U1-RESET-Pad25) -> SDA0
- U1 pad 26: unconnected-(U1-PA0/ADC0-Pad26) -> SCL0
- U1 pad 27: SIG -> A6
- U1 pad 28: TX0 -> A7
- U1 pad 29: unconnected-(U1-PA3/ADC3/RX2-Pad29) -> A8
- U1 pad 3: PREV -> TX0
- U1 pad 30: CS -> A9
- U1 pad 31: CLK -> 3V3
- U1 pad 32: MISO -> GND
- U1 pad 33: MOSI -> 5V
- U1 pad 34: unconnected-(U1-PB0/ADC8-Pad34) -> Vcc
- U1 pad 38: 3V3 -> unconnected-(U1-27_A13_SCK1-Pad38)
- U1 pad 39: GND -> unconnected-(U1-28_RX7-Pad39)
- U1 pad 4: NEXT -> unconnected-(U1-2_OUT2-Pad4)
- U1 pad 40: Vcc -> unconnected-(U1-29_TX7-Pad40)
- U1 pad 5: S0 -> unconnected-(U1-3_LRCLK2-Pad5)
- U1 pad 6: S1 -> unconnected-(U1-4_BCLK2-Pad6)
- U1 pad 7: S2 -> D5
- U1 pad 8: unconnected-(U1-PA11-Pad8) -> D6
- U1 pad 9: unconnected-(U1-PA12-Pad9) -> D7
Routing:
- net D5: track 0.00 -> 278.5 mm
- net D7: track 0.00 -> 257.8 mm
- net D6: track 0.00 -> 252.4 mm
- net D8: track 0.00 -> 250.9 mm
- net NEXT: track 208.8 -> 0.00 mm, vias 1 -> 0
- net PREV: track 198.1 -> 0.00 mm, vias 1 -> 0
- net A6: track 0.00 -> 158.7 mm
- net Net-(D2-A): track 157.3 -> 0.00 mm, vias 1 -> 0
- net pot1: track 155.2 -> 0.00 mm, vias 1 -> 0
- net ENTER: track 148.3 -> 0.00 mm, vias 1 -> 0
- net pot5: track 141.4 -> 0.00 mm, vias 2 -> 0
- net A7: track 0.00 -> 136.6 mm
- net pot2: track 135.0 -> 0.00 mm, vias 3 -> 0
- net pot6: track 124.2 -> 0.00 mm, vias 2 -> 0
- net A8: track 0.00 -> 115.3 mm
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