File: MC8P_MIDI_CONTROLLER_KiCad/MC8P_MIDI_CONTROLLER/MC8P_MIDI_CONTROLLER.kicad_sch (KiCad schematic)
At the start: 44 parts, among them J1 MIDI OUT, J2 Jack-DC, SW1 ASSIGN, SW2 ENTER, SW3 PREV, SW4 NEXT, U3 CD74HC4067M, U4 W25Q64

Commit message: PCB Updates
Parts:
- added F1: 1A_15V, Fuse:Fuse_1812_4532Metric, symbol PCM_4ms_Regulator:Polyfuse_3A_15V
Connections:
- net at C15.2, C16.1, D2.2 (A): now also F1.2; no longer J2.1
- new net: F1.1, J2.1
Other:
- moved on the sheet: C15, C16, D2
Changed lines of the file:
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@@
 	(rectangle
 		(start 133.35 128.27)
-		(end 194.31 160.02)
+		(end 209.55 160.02)
 		(stroke
 			(width 0)
@@
 	)
 	(junction
+		(at 179.07 140.97)
+		(diameter 0)
+		(color 0 0 0 0)
+	)
+	(junction
 		(at 158.75 81.28)
 		(diameter 0)
@@
 	)
 	(junction
-		(at 172.72 140.97)
+		(at 190.5 140.97)
 		(diameter 0)
 		(color 0 0 0 0)
@@
 		(color 0 0 0 0)
 	)
-	(junction
-		(at 161.29 140.97)
-		(diameter 0)
-		(color 0 0 0 0)
-	)
 	(no_connect
 		(at 120.65 127)
@@
 	(wire
 		(pts
-			(xy 161.29 147.32) (xy 161.29 148.59)
+			(xy 179.07 147.32) (xy 179.07 148.59)
 		)
 		(stroke
@@
 	(wire
 		(pts
+			(xy 170.18 140.97) (xy 179.07 140.97)
+		)
+		(stroke
+			(width 0)
+			(type default)
+		)
+	)
+	(wire
+		(pts
 			(xy 205.74 35.56) (xy 205.74 34.29)
 		)
@@
 	(wire
 		(pts
-			(xy 161.29 140.97) (xy 161.29 142.24)
+			(xy 179.07 140.97) (xy 179.07 142.24)
 		)
 		(stroke
@@
 	(wire
 		(pts
-			(xy 153.67 140.97) (xy 161.29 140.97)
-		)
-		(stroke
-			(width 0)
-			(type default)
-		)
-	)
-	(wire
-		(pts
 			(xy 158.75 80.01) (xy 158.75 81.28)
 		)
@@
 	(wire
 		(pts
-			(xy 161.29 140.97) (xy 172.72 140.97)
+			(xy 179.07 140.97) (xy 190.5 140.97)
 		)
 		(stroke
@@
 	(wire
 		(pts
-			(xy 172.72 140.97) (xy 179.07 140.97)
+			(xy 190.5 140.97) (xy 196.85 140.97)
 		)
 		(stroke
@@
 	(wire
 		(pts
+			(xy 153.67 140.97) (xy 162.56 140.97)
+		)
+		(stroke
+			(width 0)
+			(type default)
+		)
+	)
+	(wire
+		(pts
 			(xy 48.26 172.72) (xy 58.42 172.72)
 		)
@@
 	(global_label "Vcc"
 		(shape input)
-		(at 186.69 140.97 0)
+		(at 204.47 140.97 0)
 		(fields_autoplaced yes)
 		(effects
@@
 		)
 		(property "Intersheetrefs" "${INTERSHEET_REFS}"
-			(at 192.941 140.97 0)
+			(at 210.721 140.97 0)
 			(effects
 				(font
@@
 	(symbol
 		(lib_id "Device:C")
-		(at 172.72 144.78 0)
+		(at 190.5 144.78 0)
 		(unit 1)
 		(exclude_from_sim no)
@@
 		(fields_autoplaced yes)
 		(property "Reference" "C16"
-			(at 176.53 143.5099 0)
+			(at 194.31 143.5099 0)
 			(effects
 				(font
@@
 		)
 		(property "Value" "10uF"
-			(at 176.53 146.0499 0)
+			(at 194.31 146.0499 0)
 			(effects
 				(font
@@
 		)
 		(property "Footprint" "Capacitor_SMD:C_1206_3216Metric_Pad1.33x1.80mm_HandSolder"
-			(at 173.6852 148.59 0)
+			(at 191.4652 148.59 0)
 			(effects
 				(font
@@
 		)
 		(property "Datasheet" "~"
-			(at 172.72 144.78 0)
+			(at 190.5 144.78 0)
 			(effects
 				(font
@@
 		)
 		(property "Description" "Unpolarized capacitor"
-			(at 172.72 144.78 0)
+			(at 190.5 144.78 0)
 			(effects
 				(font
@@
 	(symbol
 		(lib_id "power:GND")
-		(at 172.72 148.59 0)
+		(at 190.5 148.59 0)
 		(unit 1)
 		(exclude_from_sim no)
@@
 		(fields_autoplaced yes)
 		(property "Reference" "#PWR050"
-			(at 172.72 154.94 0)
+			(at 190.5 154.94 0)
 			(effects
 				(font
@@
 		)
 		(property "Value" "GND"
-			(at 172.72 153.67 0)
+			(at 190.5 153.67 0)
 			(effects
 				(font
@@
 		)
 		(property "Footprint" ""
-			(at 172.72 148.59 0)
+			(at 190.5 148.59 0)
 			(effects
 				(font
@@
 		)
 		(property "Datasheet" ""
-			(at 172.72 148.59 0)
+			(at 190.5 148.59 0)
 			(effects
 				(font
@@
 		)
 		(property "Description" "Power symbol creates a global label with name \"GND\" , ground"
-			(at 172.72 148.59 0)
+			(at 190.5 148.59 0)
 			(effects
 				(font
@@
 	(symbol
 		(lib_id "PCM_4ms_Capacitor:100nF_0603_16V")
-		(at 161.29 144.78 180)
+		(at 179.07 144.78 180)
 		(unit 1)
 		(exclude_from_sim no)
@@
 		(fields_autoplaced yes)
 		(property "Reference" "C15"
-			(at 163.83 143.5035 0)
+			(at 181.61 143.5035 0)
 			(effects
 				(font
@@
 		)
 		(property "Value" "100nF_0603_16V"
-			(at 161.29 148.59 0)
+			(at 179.07 148.59 0)
 			(effects
 				(font
@@
 		)
 		(property "Footprint" "Capacitor_SMD:C_1206_3216Metric"
-			(at 163.83 139.7 0)
+			(at 181.61 139.7 0)
 			(effects
 				(font
@@
 		)
 		(property "Datasheet" ""
-			(at 161.29 144.78 0)
+			(at 179.07 144.78 0)
 			(effects
 				(font
@@
 		)
 		(property "Description" "0.1uF, Min. 16V 10%, X7R or X5R or similar"
-			(at 161.29 144.78 0)
+			(at 179.07 144.78 0)
 			(effects
 				(font
@@
 		)
 		(property "Specifications" "0.1uF, Min. 16V 10%, X7R or X5R or similar"
-			(at 163.83 136.906 0)
+			(at 181.61 136.906 0)
 			(effects
 				(font
@@
 		)
 		(property "Manufacturer" "AVX Corporation"
-			(at 163.83 135.382 0)
+			(at 181.61 135.382 0)
 			(effects
 				(font
@@
 		)
 		(property "Part Number" "0603YC104KAT2A"
-			(at 163.83 133.858 0)
+			(at 181.61 133.858 0)
 			(effects
 				(font
@@
 		)
 		(property "Display" "0.1uF"
-			(at 163.83 146.0435 0)
+			(at 181.61 146.0435 0)
 			(effects
 				(font
@@
 		)
 		(property "JLCPCB ID" "C14663"
-			(at 160.02 132.08 0)
+			(at 177.8 132.08 0)
 			(effects
 				(font
@@
 	(symbol
 		(lib_id "power:GND")
-		(at 161.29 148.59 0)
+		(at 179.07 148.59 0)
 		(unit 1)
 		(exclude_from_sim no)
@@
 		(fields_autoplaced yes)
 		(property "Reference" "#PWR049"
-			(at 161.29 154.94 0)
+			(at 179.07 154.94 0)
 			(effects
 				(font
@@
 		)
 		(property "Value" "GND"
-			(at 161.29 153.67 0)
+			(at 179.07 153.67 0)
 			(effects
 				(font
@@
 		)
 		(property "Footprint" ""
-			(at 161.29 148.59 0)
+			(at 179.07 148.59 0)
 			(effects
 				(font
@@
 		)
 		(property "Datasheet" ""
-			(at 161.29 148.59 0)
+			(at 179.07 148.59 0)
 			(effects
 				(font
@@
 		)
 		(property "Description" "Power symbol creates a global label with name \"GND\" , ground"
-			(at 161.29 148.59 0)
+			(at 179.07 148.59 0)
 			(effects
 				(font
@@
 	)
 	(symbol
+		(lib_id "PCM_4ms_Regulator:Polyfuse_3A_15V")
+		(at 166.37 140.97 90)
+		(unit 1)
+		(exclude_from_sim no)
+		(in_bom yes)
+		(on_board yes)
+		(dnp no)
+		(property "Reference" "F1"
+			(at 166.116 145.288 90)
+			(effects
+				(font
+					(size 1.27 1.27)
+				)
+			)
+		)
+		(property "Value" "1A_15V"
+			(at 166.116 147.828 90)
+			(effects
+				(font
+					(size 1.27 1.27)
+				)
+			)
+		)
+		(property "Footprint" "Fuse:Fuse_1812_4532Metric"
+			(at 182.88 147.32 0)
+			(effects
+				(font
+					(size 1.27 1.27)
+				)
+				(justify left)
+				(hide yes)
+			)
+		)
+		(property "Datasheet" "~"
+			(at 166.37 140.97 0)
+			(effects
+				(font
+					(size 1.27 1.27)
+				)
+				(hide yes)
+			)
+		)
+		(property "Description" "3A trip, 1.5A hold Resettable fuse, polymeric positive temperature coefficient"
+			(at 166.37 140.97 0)
+			(effects
+				(font
+					(size 1.27 1.27)
+				)
+				(hide yes)
+			)
+		)
+		(property "Specifications" "Itrip=3.0A, MaxV > 15V, 1812 package"
+			(at 179.07 140.97 0)
+			(effects
+				(font
+					(size 1.27 1.27)
+				)
+				(hide yes)
+			)
+		)
+		(property "Manufacturer" "LittleFuse"
+			(at 175.26 140.97 0)
+			(effects
+				(font
+					(size 1.27 1.27)
+				)
+				(hide yes)
+			)
+		)
+		(property "Part Number" "miniSMDC150F/24"
+			(at 177.8 140.97 0)
+			(effects
+				(font
+					(size 1.27 1.27)
+				)
+				(hide yes)
+			)
+		)
+		(property "JLCPCB ID" "C207070 "
+			(at 186.69 140.97 0)
+			(effects
+				(font
+					(size 1.27 1.27)
+				)
+				(hide yes)
+			)
+		)
+		(property "Part Number 2" "1812L150/16"
+			(at 184.15 139.7 0)
+			(effects
+				(font
+					(size 1.27 1.27)
+				)
+				(hide yes)
+			)
+		)
+		(pin "1"
+		)
+		(pin "2"
+		)
+		(instances
+			(project "MC8P_MIDI_CONTROLLER"
+				(path "/42d00d8e-48e3-47e6-b456-ac5bd2d9bc78"
+					(reference "F1")
+					(unit 1)
+				)
+			)
+		)
+	)
+	(symbol
 		(lib_id "power:GND")
 		(at 154.94 25.4 0)
@@
 	(symbol
 		(lib_id "PCM_Diode_Schottky_AKL:BAT43")
-		(at 182.88 140.97 0)
+		(at 200.66 140.97 0)
 		(unit 1)
 		(exclude_from_sim no)
@@
 		(dnp no)
 		(property "Reference" "D2"
-			(at 183.1975 134.62 0)
+			(at 200.9775 134.62 0)
 			(effects
 				(font
@@
 		)
 		(property "Value" "BAT43"
-			(at 183.1975 137.16 0)
+			(at 200.9775 137.16 0)
 			(effects
 				(font
@@
 		)
 		(property "Footprint" "Diode_SMD:D_SOD-123"
-			(at 183.388 131.572 0)
+			(at 201.168 131.572 0)
 			(effects
 				(font
@@
 		)
 		(property "Datasheet" "https://www.tme.eu/Document/1036f59816f6cf6d50674da5bd8b8c1f/BAT42.pdf"
-			(at 182.88 140.97 0)
+			(at 200.66 140.97 0)
 			(effects
 				(font
@@
 		)
 		(property "Description" "DO-35 Schottky diode, 30V, 200mA, Alternate KiCAD Library"
-			(at 182.88 140.97 0)
+			(at 200.66 140.97 0)
 			(effects
 				(font
