File: MC8P_MIDI_CONTROLLER_KiCad/MC8P_MIDI_CONTROLLER/MC8P_MIDI_CONTROLLER.kicad_sch (KiCad schematic)
At the start: 45 parts, among them J1 MIDI OUT, J2 Jack-DC, SW1 ASSIGN, SW2 ENTER, SW3 PREV, SW4 NEXT, U3 CD74HC4067M, U4 W25Q64

Commit message: Mk1 PCB
Parts:
- removed C12, C13, C14, C15: 100nF_0603_16V, Capacitor_SMD:C_1206_3216Metric, symbol PCM_4ms_Capacitor:100nF_0603_16V
- removed C16: 10uF, Capacitor_SMD:C_1206_3216Metric_Pad1.33x1.80mm_HandSolder, symbol Device:C
- removed D1: LED, LED_SMD:LED_1206_3216Metric_Pad1.42x1.75mm_HandSolder, symbol Device:LED
- removed D2: BAT43, Diode_SMD:D_SOD-123, symbol PCM_Diode_Schottky_AKL:BAT43
- removed F1: 1A_15V, Fuse:Fuse_1812_4532Metric, symbol PCM_4ms_Regulator:Polyfuse_3A_15V
- removed J2: Jack-DC, Connector_BarrelJack:BarrelJack_GCT_DCJ200-10-A_Horizontal, symbol Connector:Jack-DC
- removed R7, R8: 10k_0402, PCM_4ms_Resistor:R_0603, symbol PCM_4ms_Resistor:10k_0402
- removed U1: ~, blackpill:Z_module_black_pill_STM32F411, symbol STM32F411CEU6_BlackPill:BlackPill_STM32F411CEU6
- removed U3: CD74HC4067M, Package_SO:SOIC-24W_7.5x15.4mm_P1.27mm, symbol 74xx:CD74HC4067M
- removed U4: W25Q64, Package_SO:SOIC-8_3.9x4.9mm_P1.27mm, symbol W25Q64_SPI_FLASH:W25Q64
- added C12: 10uF_4x5.3_10V, Capacitor_THT:CP_Radial_D4.0mm_P1.50mm, symbol PCM_4ms_Capacitor:10uF_4x5.3_10V
- added J2: 5V, Connector_BarrelJack:BarrelJack_GCT_DCJ200-10-A_Horizontal, symbol Connector:Barrel_Jack_MountingPin
- added U1: Teensy4.0, teensy:Teensy40, symbol teensy:Teensy4.0
- C1, C2, C3, C4, C5, C6, C7, C8: footprint Capacitor_SMD:C_1206_3216Metric_Pad1.33x1.80mm_HandSolder -> Capacitor_THT:C_Axial_L3.8mm_D2.6mm_P7.50mm_Horizontal
- C10, C9: footprint Capacitor_SMD:C_1206_3216Metric_Pad1.33x1.80mm_HandSolder -> Capacitor_THT:C_Disc_D5.0mm_W2.5mm_P5.00mm
- R1, R2, R3, R4: footprint PCM_4ms_Resistor:R_0603 -> PCM_4ms_Resistor:R_Axial_DIN0207_L6.3mm_D2.5mm_P7.62mm_Horizontal
- R5, R6: footprint PCM_4ms_Resistor:R_0603 -> PCM_4ms_Resistor:R_Axial_DIN0207_L6.3mm_D2.5mm_P7.62mm_Horizontal; Display 33R -> 220R
- renumbered SSD1306 to SSD1
Connections:
- net 3V3: now also U1.31 (3V3); no longer R6.1
- net GND: now also C12.2, J2.2, J2.MP (MountPin), U1.1 (GND), U1.17 (GND), U1.32 (GND), U1.47 (GND)
- net SCL0: now also U1.26 (19_A5_SCL0)
- net SDA0: now also U1.25 (18_A4_SDA0)
- net TX0: now also U1.3 (1_TX1_CTX2_MISO1)
- net Vcc: now also R6.1, U1.34 (VUSB)
- net ASSIGN renamed D5
- net D5: now also U1.7 (5_IN2)
- net ENTER renamed D6
- net D6: now also U1.8 (6_OUT1D)
- net NEXT renamed D8
- net D8: now also U1.10 (8_TX2_IN1)
- net PREV renamed D7
- net D7: now also U1.9 (7_RX2_OUT1A)
- net pot1 renamed A0
- net A0: now also U1.21 (14_A0_TX3_SPDIF_OUT)
- net pot2 renamed A1
- net A1: now also U1.22 (15_A1_RX3_SPDIF_IN)
- net pot3 renamed A2
- net A2: now also U1.23 (16_A2_RX4_SCL1)
- net pot4 renamed A3
- net A3: now also U1.24 (17_A3_TX4_SDA1)
- net pot5 renamed A6
- net A6: now also C8.1, U1.27 (20_A6_TX5_LRCLK1); no longer C5.1
- net pot6 renamed A7
- net A7: now also C7.1, U1.28 (21_A7_RX5_BCLK1); no longer C6.1
- net pot7 renamed A8
- net A8: now also C6.1, U1.29 (22_A8_CTX1); no longer C7.1
- net pot8 renamed A9
- net A9: now also C5.1, U1.30 (23_A9_CRX1_MCLK1); no longer C8.1
- new net 5V: C12.1, J2.1, U1.33 (VIN)
- no-connect marks 8 -> 32
Other:
- note added: "5V DC in"
- note added: "teensy"
- note removed: "5V DC Input"
- note removed: "FLASH MEMORY"
- note removed: "MUX"
- note removed: "STM32F411CEU6 Blackpill"
- moved on the sheet: C1, C10, C11, C2, C3, C4, C5, C6, C7, C8, C9, J1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
